File: Drone_FC_project.kicad_sch (KiCad schematic)
At the start: 34 parts, among them J5 Battery_pins, J6 USB_C_Receptacle, SW2 SW_Push, U3 AP2112K-3.3TRG1, U4 STM32F411CEU6, Y1 X322516MOB4SI

Commit message: footprints and spacing
Added half the footprints and made thigns look nicer.
Parts:
- C1, C11, C12, C13, C16, C2, C3, C4: footprint Capacitor_SMD:C_0603_1608Metric -> Capacitor_SMD:C_0402_1005Metric
- C10, C9: footprint Package_TO_SOT_SMD:SOT-23-5 -> Capacitor_SMD:C_0603_1608Metric
- C14, C5, C6: footprint Package_SO:SOIC-8_3.9x4.9mm_P1.27mm -> Capacitor_SMD:C_0603_1608Metric
- C22: footprint Package_SO:SOIC-8_3.9x4.9mm_P1.27mm -> Capacitor_SMD:C_0805_2012Metric
- C7: footprint Package_SO:SOIC-8_3.9x4.9mm_P1.27mm -> Capacitor_SMD:C_0402_1005Metric
- R10, R11, R12, R14, R16, R9: footprint (none) -> Resistor_SMD:R_0402_1005Metric
- R13: footprint Package_TO_SOT_SMD:SOT-23 -> Resistor_SMD:R_0402_1005Metric
Changed lines of the file:
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@@
 	(rectangle
 		(start 15.24 15.24)
-		(end 199.39 124.46)
+		(end 190.5 124.46)
+		(stroke
+			(width 0)
+			(type default)
+		)
+		(fill
+			(type none)
+		)
+	)
+	(rectangle
+		(start 157.48 21.59)
+		(end 184.15 50.8)
 		(stroke
 			(width 0)
@@
 	(wire
 		(pts
-			(xy 143.51 40.64) (xy 148.59 40.64)
+			(xy 143.51 41.91) (xy 162.56 41.91)
 		)
 		(stroke
@@
 	(wire
 		(pts
-			(xy 143.51 49.53) (xy 143.51 40.64)
+			(xy 143.51 49.53) (xy 143.51 41.91)
 		)
 		(stroke
@@
 	(wire
 		(pts
-			(xy 140.97 36.83) (xy 148.59 36.83)
+			(xy 140.97 38.1) (xy 162.56 38.1)
 		)
 		(stroke
@@
 	(wire
 		(pts
-			(xy 135.89 29.21) (xy 148.59 29.21)
+			(xy 135.89 30.48) (xy 162.56 30.48)
 		)
 		(stroke
@@
 	(wire
 		(pts
-			(xy 138.43 33.02) (xy 148.59 33.02)
+			(xy 138.43 34.29) (xy 162.56 34.29)
 		)
 		(stroke
@@
 	(wire
 		(pts
-			(xy 140.97 46.99) (xy 140.97 36.83)
+			(xy 140.97 46.99) (xy 140.97 38.1)
 		)
 		(stroke
@@
 	(wire
 		(pts
-			(xy 138.43 44.45) (xy 138.43 33.02)
+			(xy 138.43 44.45) (xy 138.43 34.29)
 		)
 		(stroke
@@
 	(wire
 		(pts
-			(xy 135.89 41.91) (xy 135.89 29.21)
+			(xy 135.89 41.91) (xy 135.89 30.48)
 		)
 		(stroke
@@
 			)
 		)
-		(property "Footprint" "Package_SO:SOIC-8_3.9x4.9mm_P1.27mm"
+		(property "Footprint" "Capacitor_SMD:C_0402_1005Metric"
 			(at 42.8752 30.48 0)
 			(hide yes)
@@
 		(in_pos_files yes)
 		(dnp no)
-		(fields_autoplaced yes)
 		(property "Reference" "D5"
 			(at 85.09 152.7174 90)
@@
 		)
 		(property "Value" "GREEN"
-			(at 85.09 155.2574 90)
+			(at 84.582 155.194 90)
 			(show_name no)
 			(do_not_autoplace no)
@@
 			)
 		)
-		(property "Footprint" ""
+		(property "Footprint" "Resistor_SMD:R_0402_1005Metric"
 			(at 120.142 152.4 90)
 			(hide yes)
@@
 			)
 		)
-		(property "Footprint" ""
+		(property "Footprint" "Resistor_SMD:R_0402_1005Metric"
 			(at 120.142 165.1 90)
 			(hide yes)
@@
 			)
 		)
-		(property "Footprint" "Package_SO:SOIC-8_3.9x4.9mm_P1.27mm"
+		(property "Footprint" "Capacitor_SMD:C_0603_1608Metric"
 			(at 31.4452 30.48 0)
 			(hide yes)
@@
 			)
 		)
-		(property "Footprint" "Capacitor_SMD:C_0603_1608Metric"
+		(property "Footprint" "Capacitor_SMD:C_0402_1005Metric"
 			(at 70.8152 30.48 0)
 			(hide yes)
@@
 			)
 		)
-		(property "Footprint" ""
+		(property "Footprint" "Resistor_SMD:R_0402_1005Metric"
 			(at 99.822 162.56 90)
 			(hide yes)
@@
 			)
 		)
-		(property "Footprint" ""
+		(property "Footprint" "Resistor_SMD:R_0402_1005Metric"
 			(at 210.312 142.24 90)
 			(hide yes)
@@
 			)
 		)
-		(property "Footprint" "Capacitor_SMD:C_0603_1608Metric"
+		(property "Footprint" "Capacitor_SMD:C_0402_1005Metric"
 			(at 79.7052 30.48 0)
 			(hide yes)
@@
 			)
 		)
-		(property "Footprint" "Package_SO:SOIC-8_3.9x4.9mm_P1.27mm"
+		(property "Footprint" "Capacitor_SMD:C_0603_1608Metric"
 			(at 74.6252 118.11 0)
 			(hide yes)
@@
 			)
 		)
-		(property "Footprint" "Package_SO:SOIC-8_3.9x4.9mm_P1.27mm"
+		(property "Footprint" "Capacitor_SMD:C_0603_1608Metric"
 			(at 119.0752 30.48 0)
 			(hide yes)
@@
 			)
 		)
-		(property "Footprint" "Package_TO_SOT_SMD:SOT-23-5"
+		(property "Footprint" "Capacitor_SMD:C_0603_1608Metric"
 			(at 55.5752 168.91 0)
 			(hide yes)
@@
 			)
 		)
-		(property "Footprint" "Capacitor_SMD:C_0603_1608Metric"
+		(property "Footprint" "Capacitor_SMD:C_0402_1005Metric"
 			(at 46.6852 43.18 0)
 			(hide yes)
@@
 		(in_pos_files yes)
 		(dnp no)
-		(fields_autoplaced yes)
 		(property "Reference" "D6"
 			(at 105.41 152.7174 90)
@@
 		)
 		(property "Value" "GREEN"
-			(at 105.41 155.2574 90)
+			(at 104.902 155.194 90)
 			(show_name no)
 			(do_not_autoplace no)
@@
 			)
 		)
-		(property "Footprint" "Package_TO_SOT_SMD:SOT-23"
+		(property "Footprint" "Resistor_SMD:R_0402_1005Metric"
 			(at 58.42 47.752 90)
 			(hide yes)
@@
 			)
 		)
-		(property "Footprint" ""
+		(property "Footprint" "Resistor_SMD:R_0402_1005Metric"
 			(at 217.932 142.24 90)
 			(hide yes)
@@
 			)
 		)
-		(property "Footprint" "Capacitor_SMD:C_0603_1608Metric"
+		(property "Footprint" "Capacitor_SMD:C_0402_1005Metric"
 			(at 53.0352 30.48 0)
 			(hide yes)
@@
 			)
 		)
-		(property "Footprint" "Capacitor_SMD:C_0603_1608Metric"
+		(property "Footprint" "Capacitor_SMD:C_0402_1005Metric"
 			(at 50.4952 82.55 0)
 			(hide yes)
@@
 			)
 		)
-		(property "Footprint" "Capacitor_SMD:C_0603_1608Metric"
+		(property "Footprint" "Capacitor_SMD:C_0402_1005Metric"
 			(at 110.1852 30.48 0)
 			(hide yes)
@@
 			)
 		)
-		(property "Footprint" "Capacitor_SMD:C_0603_1608Metric"
+		(property "Footprint" "Capacitor_SMD:C_0402_1005Metric"
 			(at 32.7152 82.55 0)
 			(hide yes)
@@
 			)
 		)
-		(property "Footprint" "Capacitor_SMD:C_0603_1608Metric"
+		(property "Footprint" "Capacitor_SMD:C_0402_1005Metric"
 			(at 61.9252 30.48 0)
 			(hide yes)
@@
 			)
 		)
-		(property "Footprint" ""
+		(property "Footprint" "Resistor_SMD:R_0402_1005Metric"
 			(at 79.502 162.56 90)
 			(hide yes)
@@
 			)
 		)
-		(property "Footprint" "Package_SO:SOIC-8_3.9x4.9mm_P1.27mm"
+		(property "Footprint" "Capacitor_SMD:C_0805_2012Metric"
 			(at 24.4348 157.48 0)
 			(hide yes)
@@
 			)
 		)
-		(property "Footprint" "Package_TO_SOT_SMD:SOT-23-5"
+		(property "Footprint" "Capacitor_SMD:C_0603_1608Metric"
 			(at 30.1752 168.91 0)
 			(hide yes)
@@
 	)
 	(sheet
-		(at 148.59 25.4)
+		(at 162.56 26.67)
 		(size 16.51 19.05)
 		(exclude_from_sim no)
@@
 		)
 		(property "Sheetname" "Motors"
-			(at 148.59 24.6884 0)
+			(at 162.56 25.9584 0)
 			(show_name no)
 			(do_not_autoplace no)
@@
 		)
 		(property "Sheetfile" "Motors.kicad_sch"
-			(at 145.034 45.212 0)
+			(at 159.004 46.482 0)
 			(show_name no)
 			(do_not_autoplace no)
@@
 		)
 		(pin "MOTOR 1" input
-			(at 148.59 29.21 180)
+			(at 162.56 30.48 180)
 			(effects
 				(font
@@
 		)
 		(pin "MOTOR 2" input
-			(at 148.59 33.02 180)
+			(at 162.56 34.29 180)
 			(effects
 				(font
@@
 		)
 		(pin "MOTOR 3" input
-			(at 148.59 36.83 180)
+			(at 162.56 38.1 180)
 			(effects
 				(font
@@
 		)
 		(pin "MOTOR 4" input
-			(at 148.59 40.64 180)
+			(at 162.56 41.91 180)
 			(effects
 				(font
