File: Battery_and_regulator.kicad_sch (KiCad schematic)
At the start: 0 parts

Commit message: Finished motor and battery/regulator subfolders
Also made a folder for holding datasheets.
Parts:
- added C1, C2: 1u, Package_TO_SOT_SMD:SOT-23-5, symbol Device:C
- added D5: LED, symbol Device:LED
- added J5: Conn_01x04_Pin, Package_DIP:DIP-6_W7.62mm, symbol Connector:Conn_01x04_Pin
- added R9: 1k, symbol Device:R
- added U3: AP2112K-3.3TRG1, Package_TO_SOT_SMD:SOT-23-5, symbol Regulator_Linear:AP2112K-3.3
Connections:
- new net: D5.1 (K), R9.1
- new net +3.3V: C2.1, D5.2 (A), U3.5 (VOUT)
- new net +BATT: C1.1, J5.1 (Pin_1), J5.2 (Pin_2), U3.1 (VIN), U3.3 (EN)
- new net GND: C1.2, C2.2, J5.3 (Pin_3), J5.4 (Pin_4), R9.2, U3.2 (GND)
Other:
- note added: "Capacitors based off of manufacturer's datasheet"
- note added: "RED LED To inidicate 3.3V is running"
- note added: "The pins that attach to the battery"
- note added: "Tie EN to HIGH"
- note added: "We could take this sublevel folder out later bc it has no inputs and outputs"
- title: (none) -> Battery and Regulator
