File: Battery_and_regulator.kicad_sch (KiCad schematic)
At the start: 6 parts, among them J5 Conn_01x04_Pin, U3 AP2112K-3.3TRG1

Commit message: Updated stm32
Updated stm32 and usb-c
Parts:
- removed C1, C2: 1u, Package_TO_SOT_SMD:SOT-23-5, symbol Device:C
- removed D5: LED, symbol Device:LED
- removed J5: Conn_01x04_Pin, Package_DIP:DIP-6_W7.62mm, symbol Connector:Conn_01x04_Pin
- removed R9: 1k, symbol Device:R
- removed U3: AP2112K-3.3TRG1, Package_TO_SOT_SMD:SOT-23-5, symbol Regulator_Linear:AP2112K-3.3
Other:
- note removed: "Capacitors based off of manufacturer's datasheet"
- note removed: "RED LED To inidicate 3.3V is running"
- note removed: "The pins that attach to the battery"
- note removed: "Tie EN to HIGH"
- note removed: "We could take this sublevel folder out later bc it has no inputs and outputs"
