File: imu.kicad_sch (KiCad schematic)
At the start: 1 part, among them U1 BMI088

Commit message: IMU
Parts:
- added C3: 100n, Package_LGA:Bosch_LGA-16_4.5x3mm_P0.5mm_LayoutBorder7x1y_ClockwisePinNumbering, symbol Device:C
Connections:
- net INT_GYR: now reaches U1.1 (INT2)
- net INT_GYR: now also U1.12 (INT3)
- net VCCA: now reaches U1.10 (SDO2)
- net VCCA: now also U1.11 (VDDIO), U1.3 (VDD), U1.7 (PS), C3.1
- net GND: now reaches U1.15 (SDO1)
- net GND: now also U1.2 (GNDA), U1.4 (GNDA), U1.6 (GNDIO), C3.2
- net INT_ACC: now reaches U1.16 (INT1)
- net IMU_SCL: now reaches U1.8 (SCK/SCL)
- net IMU_SDA: now reaches U1.9 (SDI/SDA)
- no-connect marks 0 -> 3
