File: Motors.kicad_sch (KiCad schematic)
At the start: 20 parts, among them J1 Conn_01x02_Pin, J2 Conn_01x02_Pin, J3 Conn_01x02_Pin, J4 Conn_01x02_Pin, Q1 AO3400A, Q2 AO3400A, Q3 AO3400A, Q4 AO3400A

Commit message: updated pin to accurate size
Parts:
- J1, J2, J3, J4: footprint Connector_AMASS:AMASS_XT30PW-F_1x02_P2.50mm_Horizontal -> Connector_JST:JST_SH_BM02B-SRSS-TB_1x02-1MP_P1.00mm_Vertical
- R1: footprint (none) -> Connector_JST:JST_SH_BM02B-SRSS-TB_1x02-1MP_P1.00mm_Vertical
Changed lines of the file:
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@@
 			)
 		)
-		(property "Footprint" "Connector_AMASS:AMASS_XT30PW-F_1x02_P2.50mm_Horizontal"
+		(property "Footprint" "Connector_JST:JST_SH_BM02B-SRSS-TB_1x02-1MP_P1.00mm_Vertical"
 			(at 124.46 59.69 0)
 			(hide yes)
@@
 			)
 		)
-		(property "Footprint" "Connector_AMASS:AMASS_XT30PW-F_1x02_P2.50mm_Horizontal"
+		(property "Footprint" "Connector_JST:JST_SH_BM02B-SRSS-TB_1x02-1MP_P1.00mm_Vertical"
 			(at 124.46 120.65 0)
 			(hide yes)
@@
 			)
 		)
-		(property "Footprint" "Connector_AMASS:AMASS_XT30PW-F_1x02_P2.50mm_Horizontal"
+		(property "Footprint" "Connector_JST:JST_SH_BM02B-SRSS-TB_1x02-1MP_P1.00mm_Vertical"
 			(at 222.25 121.92 0)
 			(hide yes)
@@
 			)
 		)
-		(property "Footprint" "Connector_AMASS:AMASS_XT30PW-F_1x02_P2.50mm_Horizontal"
+		(property "Footprint" "Connector_JST:JST_SH_BM02B-SRSS-TB_1x02-1MP_P1.00mm_Vertical"
 			(at 222.25 59.69 0)
 			(hide yes)
@@
 			)
 		)
-		(property "Footprint" ""
+		(property "Footprint" "Connector_JST:JST_SH_BM02B-SRSS-TB_1x02-1MP_P1.00mm_Vertical"
 			(at 95.25 75.438 90)
 			(hide yes)

Commit message: IMU, VBAT_Sense,
Fixed some decoupling issues, made the IMU into SPI mode. Wired all to stm32. Few updates on the appearances as well to make it look more organized.
Changed lines of the file:
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@@
 		(property "Value" "GND"
 			(at 114.3 92.71 0)
+			(hide yes)
 			(show_name no)
 			(do_not_autoplace no)
@@
 		(property "Value" "GND"
 			(at 114.3 153.67 0)
+			(hide yes)
 			(show_name no)
 			(do_not_autoplace no)
@@
 		(property "Value" "GND"
 			(at 212.09 92.71 0)
+			(hide yes)
 			(show_name no)
 			(do_not_autoplace no)
@@
 		(property "Value" "GND"
 			(at 212.09 154.94 0)
-			(show_name no)
-			(do_not_autoplace no)
+			(hide yes)
+			(show_name no)
+			(do_not_autoplace no)

Commit message: Motor and UBS 5V update
Motors each have a RED LED to indicate their on status.
5V on USB now runs when and only when the USB is plugged in. It will ignore battery otherwise. Green Led's indicate if the power is running.
Parts:
- removed R7: 47R, symbol Device:R
- added D10, D7, D8, D9: RED, symbol Device:LED
- added R17, R19, R20, R21: 1k, symbol Device:R
- added R18: 47R, Connector_JST:JST_SH_BM02B-SRSS-TB_1x02-1MP_P1.00mm_Vertical, symbol Device:R
- R3, R5: footprint (none) -> Connector_JST:JST_SH_BM02B-SRSS-TB_1x02-1MP_P1.00mm_Vertical
Connections:
- net GND: now also R17.2, R19.2, R20.2, R21.2
- net MOTOR 3: now also R18.1; no longer R5.1
- net MOTOR 4: now also R5.1
- net at Q1.1 (G), R1.2, R2.1: now also D7.2 (A)
- net at Q2.1 (G), R3.2, R4.1: now also D10.2 (A)
- net at Q4.1 (G), R8.1: now also R5.2, D9.2 (A)
- net at Q3.1 (G), R6.1: now also D8.2 (A), R18.2; no longer R5.2
- new net: D8.1 (K), R19.1
- new net: D10.1 (K), R21.1
- new net: D9.1 (K), R20.1
- new net: D7.1 (K), R17.1
Other:
- note removed: "Pull Down Resistor"
- moved on the sheet: R1

Commit message: footprints and spacing
Added half the footprints and made thigns look nicer.
Parts:
- R1, R18, R3, R5: footprint Connector_JST:JST_SH_BM02B-SRSS-TB_1x02-1MP_P1.00mm_Vertical -> Resistor_SMD:R_0402_1005Metric
- R17, R19, R2, R20, R21, R4, R6, R8: footprint (none) -> Resistor_SMD:R_0402_1005Metric
Changed lines of the file:
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@@
 			)
 		)
-		(property "Footprint" ""
+		(property "Footprint" "Resistor_SMD:R_0402_1005Metric"
 			(at 93.472 147.32 90)
 			(hide yes)
@@
 			)
 		)
-		(property "Footprint" "Connector_JST:JST_SH_BM02B-SRSS-TB_1x02-1MP_P1.00mm_Vertical"
+		(property "Footprint" "Resistor_SMD:R_0402_1005Metric"
 			(at 88.9 136.398 90)
 			(hide yes)
@@
 			)
 		)
-		(property "Footprint" ""
+		(property "Footprint" "Resistor_SMD:R_0402_1005Metric"
 			(at 198.882 143.51 90)
 			(hide yes)
@@
 			)
 		)
-		(property "Footprint" ""
+		(property "Footprint" "Resistor_SMD:R_0402_1005Metric"
 			(at 101.092 81.28 90)
 			(hide yes)
@@
 			)
 		)
-		(property "Footprint" ""
+		(property "Footprint" "Resistor_SMD:R_0402_1005Metric"
 			(at 191.262 86.36 90)
 			(hide yes)
@@
 			)
 		)
-		(property "Footprint" ""
+		(property "Footprint" "Resistor_SMD:R_0402_1005Metric"
 			(at 101.092 142.24 90)
 			(hide yes)
@@
 			)
 		)
-		(property "Footprint" ""
+		(property "Footprint" "Resistor_SMD:R_0402_1005Metric"
 			(at 191.262 148.59 90)
 			(hide yes)
@@
 			)
 		)
-		(property "Footprint" "Connector_JST:JST_SH_BM02B-SRSS-TB_1x02-1MP_P1.00mm_Vertical"
+		(property "Footprint" "Resistor_SMD:R_0402_1005Metric"
 			(at 186.69 75.438 90)
 			(hide yes)
@@
 			)
 		)
-		(property "Footprint" ""
+		(property "Footprint" "Resistor_SMD:R_0402_1005Metric"
 			(at 198.882 81.28 90)
 			(hide yes)
@@
 			)
 		)
-		(property "Footprint" "Connector_JST:JST_SH_BM02B-SRSS-TB_1x02-1MP_P1.00mm_Vertical"
+		(property "Footprint" "Resistor_SMD:R_0402_1005Metric"
 			(at 88.9 75.438 90)
 			(hide yes)
@@
 			)
 		)
-		(property "Footprint" ""
+		(property "Footprint" "Resistor_SMD:R_0402_1005Metric"
 			(at 93.472 86.36 90)
 			(hide yes)
@@
 			)
 		)
-		(property "Footprint" "Connector_JST:JST_SH_BM02B-SRSS-TB_1x02-1MP_P1.00mm_Vertical"
+		(property "Footprint" "Resistor_SMD:R_0402_1005Metric"
 			(at 186.69 137.668 90)
 			(hide yes)

Commit message: more footprint work and downloaded some
Parts:
- removed J1, J2, J3, J4: Conn_01x02_Pin, Connector_JST:JST_SH_BM02B-SRSS-TB_1x02-1MP_P1.00mm_Vertical, symbol Connector:Conn_01x02_Pin
- added J1, J2, J3, J4: Conn_01x02_MountingPin, Connector_JST:JST_SH_BM02B-SRSS-TB_1x02-1MP_P1.00mm_Vertical, symbol Connector_Generic_MountingPin:Conn_01x02_MountingPin
- D1, D2, D3, D4: footprint Diode_SMD:D_SMA -> drone_libary:SS14
- D10, D7, D8, D9: footprint (none) -> LED_SMD:LED_0603_1608Metric
- Q1, Q2, Q3, Q4: footprint Package_TO_SOT_SMD:SOT-23 -> drone_libary:SOT-23-3_AO3400A
Connections:
- net +BATT: now also J1.1 (Pin_1), J2.1 (Pin_1), J3.1 (Pin_1), J4.1 (Pin_1)
- net GND: now also J1.MP (MountPin), J2.MP (MountPin), J3.MP (MountPin), J4.MP (MountPin)
- net at D1.2 (A), Q1.3 (D): now also J1.2 (Pin_2)
- net at D2.2 (A), Q2.3 (D): now also J2.2 (Pin_2)
- net at D3.2 (A), Q3.3 (D): now also J3.2 (Pin_2)
- net at D4.2 (A), Q4.3 (D): now also J4.2 (Pin_2)
